File: choc-keyboard.kicad_pcb (KiCad board)
At the start: 2 copper layers, 35.5 x 14 mm, 77 parts, among them U1 AdafruitCharli, U2 BlackPill

Commit message: updated footprints
M  .gitignore
M  choc-keyboard.kicad_pcb
M  choc-keyboard.kicad_prl
M  choc-keyboard.kicad_pro
M  choc-keyboard.kicad_sch
M  placesw.py
A  switch-plate/.gitignore
A  switch-plate/Kailh.kicad_sym
A  switch-plate/fp-lib-table
A  switch-plate/kailh-local.kicad_sym
A  switch-plate/switch-plate.kicad_pcb
A  switch-plate/switch-plate.kicad_prl
A  switch-plate/switch-plate.kicad_pro
A  switch-plate/switch-plate.kicad_sch
A  switch-plate/sym-lib-table
A  top-plate/.gitignore
A  top-plate/fp-lib-table
A  top-plate/kailh.pretty/AdafruitCharliplex.kicad_mod
A  top-plate/kailh.pretty/BlackPill_STLINK.kicad_mod
A  top-plate/kailh.pretty/SW_Kailh_Choc_Cutout.kicad_mod
A  top-plate/sym-lib-table
A  top-plate/top-plate.kicad_pcb
A  top-plate/top-plate.kicad_prl
A  top-plate/top-plate.kicad_pro
A  top-plate/top-plate.kicad_sch
Parts:
- added H1: MountingHole, blackpill:MountingHole_2.2mm_M2_jlcpcb, F.Cu at (9.50, 15.3)
- added H10: MountingHole, blackpill:MountingHole_2.2mm_M2_jlcpcb, F.Cu at (230.4, 87.3)
- added H11: MountingHole, blackpill:MountingHole_2.2mm_M2_jlcpcb, F.Cu at (270.8, 87.3)
- added H12: MountingHole, blackpill:MountingHole_2.2mm_M2_jlcpcb, F.Cu at (258.9, 51.3)
- added H13: MountingHole, blackpill:MountingHole_2.2mm_M2_jlcpcb, F.Cu at (225.6, 65.7)
- added H14: MountingHole, blackpill:MountingHole_2.2mm_M2_jlcpcb, F.Cu at (194.8, 51.3)
- added H15: MountingHole, blackpill:MountingHole_2.2mm_M2_jlcpcb, F.Cu at (156.8, 51.3)
- added H16: MountingHole, blackpill:MountingHole_2.2mm_M2_jlcpcb, F.Cu at (118.8, 51.3)
- added H17: MountingHole, blackpill:MountingHole_2.2mm_M2_jlcpcb, F.Cu at (42.8, 51.3)
- added H18: MountingHole, kailh-choc:TestPoint_Plated_Hole_D1.2mm, F.Cu at (28.5, 15.3)
- added H19: MountingHole, kailh-choc:TestPoint_Plated_Hole_D1.2mm, F.Cu at (104.5, 15.3)
- added H2: MountingHole, blackpill:MountingHole_2.2mm_M2_jlcpcb, F.Cu at (66.5, 15.3)
- added H20: MountingHole, kailh-choc:TestPoint_Plated_Hole_D1.2mm, F.Cu at (218.5, 15.3)
- added H21: MountingHole, kailh-choc:TestPoint_Plated_Hole_D1.2mm, F.Cu at (235.1, 51.3)
- added H22: MountingHole, kailh-choc:TestPoint_Plated_Hole_D1.2mm, F.Cu at (230.4, 94.5)
- added H23: MountingHole, kailh-choc:TestPoint_Plated_Hole_D1.2mm, F.Cu at (140.6, 83.7)
- added H24: MountingHole, kailh-choc:TestPoint_Plated_Hole_D1.2mm, F.Cu at (0.00, 89.1)
- added H25: MountingHole, kailh-choc:TestPoint_Plated_Hole_D1.2mm, F.Cu at (61.8, 54.0)
- added H3: MountingHole, blackpill:MountingHole_2.2mm_M2_jlcpcb, F.Cu at (123.5, 15.3)
- added H4: MountingHole, blackpill:MountingHole_2.2mm_M2_jlcpcb, F.Cu at (180.5, 15.3)
- added H5: MountingHole, blackpill:MountingHole_2.2mm_M2_jlcpcb, F.Cu at (237.5, 15.3)
- added H6: MountingHole, blackpill:MountingHole_2.2mm_M2_jlcpcb, F.Cu at (9.88, 79.2)
- added H7: MountingHole, blackpill:MountingHole_2.2mm_M2_jlcpcb, F.Cu at (38.0, 87.3)
- added H8: MountingHole, blackpill:MountingHole_2.2mm_M2_jlcpcb, F.Cu at (82.8, 90.9)
- added H9: MountingHole, blackpill:MountingHole_2.2mm_M2_jlcpcb, F.Cu at (147.2, 83.7)
- U2: value BlackPill -> BlackPill_STLINK
Connections:
- U2 pad 5: unconnected-(U2-Pad5) -> /C14
- U2 pad 7: /C14 -> unconnected-(U2-Pad7)
Routing:
- net CA3: track 484.4 -> 473.5 mm, vias 42 -> 38
- net CA8: track 414.5 -> 421.3 mm
- net CA9: track 367.0 -> 372.7 mm, vias 18 -> 17
- net /C14: track 348.0 -> 353.1 mm
- net CA2: track 471.2 -> 466.5 mm, vias 34 -> 33
- net CA4: track 455.2 -> 459.6 mm, vias 24 -> 22
- net /R3: track 327.1 -> 330.0 mm, vias 0 -> 2
- net CA6: track 494.2 -> 497.0 mm
- net CA5: track 514.2 -> 516.7 mm
- net /C5: track 162.5 -> 164.6 mm, vias 3 -> 4
- net CA7: track 461.9 -> 463.9 mm
- net /C4: track 156.2 -> 154.2 mm
- net GND: track 106.7 -> 108.5 mm
- net /R5: track 383.8 -> 384.7 mm, vias 6 -> 8
- net Net-(U1-Pad14): track 103.9 -> 104.7 mm
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Other:
- board size 35.5 x 14 mm -> 311.9 x 106 mm
