File: choc-keyboard.kicad_sch (KiCad schematic)
At the start: 77 parts, among them U1 AdafruitCharli, U2 BlackPill_STLINK

Commit message: updated footprints
M  .gitignore
M  choc-keyboard.kicad_pcb
M  choc-keyboard.kicad_prl
M  choc-keyboard.kicad_pro
M  choc-keyboard.kicad_sch
M  placesw.py
A  switch-plate/.gitignore
A  switch-plate/Kailh.kicad_sym
A  switch-plate/fp-lib-table
A  switch-plate/kailh-local.kicad_sym
A  switch-plate/switch-plate.kicad_pcb
A  switch-plate/switch-plate.kicad_prl
A  switch-plate/switch-plate.kicad_pro
A  switch-plate/switch-plate.kicad_sch
A  switch-plate/sym-lib-table
A  top-plate/.gitignore
A  top-plate/fp-lib-table
A  top-plate/kailh.pretty/AdafruitCharliplex.kicad_mod
A  top-plate/kailh.pretty/BlackPill_STLINK.kicad_mod
A  top-plate/kailh.pretty/SW_Kailh_Choc_Cutout.kicad_mod
A  top-plate/sym-lib-table
A  top-plate/top-plate.kicad_pcb
A  top-plate/top-plate.kicad_prl
A  top-plate/top-plate.kicad_pro
A  top-plate/top-plate.kicad_sch
Parts:
- added H1, H10, H11, H12, H13, H14, H15, H16, H17, H2, H3, H4, H5, H6, H7, H8, H9: MountingHole, blackpill:MountingHole_2.2mm_M2_jlcpcb, symbol Mechanical:MountingHole
- added H18, H19, H20, H21, H22, H23, H24, H25: MountingHole, kailh-choc:TestPoint_Plated_Hole_D1.2mm, symbol Mechanical:MountingHole
Connections:
- net C14: now also U2.5 (PA8); no longer U2.7 (PA10)
